Commit message: [mycobot_description] add inertia to each links of mycobot_urdf.urdf

File: mycobot_description/urdf/mycobot/mycobot_urdf.urdf (robot description, URDF)
Before this commit: robot firefighter, 7 links, 6 joints
Links:
- link joint1: mass None -> 10
- link joint2: mass None -> 0.2
- link joint3: mass None -> 0.2
- link joint4: mass None -> 0.2
- link joint5: mass None -> 0.2
- link joint6: mass None -> 0.2
- link joint6_flange: mass None -> 0.1
